File: PCB/WateringSystem_PCB/WateringSystem_PCB.kicad_sch (KiCad schematic)
At the start: 47 parts, among them J2_SOLAR1 Conn_01x02, J3_MoistureSensor1 Conn_01x04, J4_BUTTON1 Conn_01x02, J5_LEDS1 Conn_01x08, J6_PUMP1 Conn_01x02, J7_BATT1 Conn_01x02, Q1 AO3400A, U1 TP4056-42-ESOP8, U2 MT3608

Commit message: Add decoupling capacitors on 5V and 3V3
Parts:
- added C6, C7: 100nF, Capacitor_SMD:C_1206_3216Metric_Pad1.33x1.80mm_HandSolder, symbol Device:C
Connections:
- net +5V: now also C6.2
- net GND: now also C6.1, C7.2
- net at ESP32-C3_SuperMini1.11 (3V3), J3_MoistureSensor1.4 (Pin_4), J4_BUTTON1.1 (Pin_1): now also C7.1
