File: PCB/WateringSystem_PCB/WateringSystem_PCB.kicad_sch (KiCad schematic)
At the start: 49 parts, among them J2_SOLAR1 Conn_01x02, J3_MoistureSensor1 Conn_01x04, J4_BUTTON1 Conn_01x02, J5_LEDS1 Conn_01x08, J6_PUMP1 Conn_01x02, J7_BATT1 Conn_01x02, Q1 AO3400A, U1 TP4056-42-ESOP8, U2 MT3608

Commit message: Fix errors in pcb design.
Connections:
- net MOISTURE_SENSOR_ANALOG: now also ESP32-C3_SuperMini1.15 (GPIO1), J3_MoistureSensor1.1 (Pin_1)
- net +5V: no longer names the net of C6.2, ESP32-C3_SuperMini1.9 (5V), R_LED1.2, R_LED2.2, R_LED3.2, R_LED4.2, TP_5V1.1
- net +5V: no longer C4.1, L1.2, Q1.3 (D), R4.1, R6.2, U2.1 (SW)
- net +V_PUMP: no longer names the net of D1.1 (K), J6_PUMP1.2 (Pin_2), TP_PUMP1.1
- net +V_PUMP: no longer Q1.2 (S)
- net +V_SOL: no longer names the net of R_SOL1.1, TP_VSOL1.1
- net +V_SOL: no longer J2_SOLAR1.2 (Pin_2), R1.1
- net TP4056_VCC: no longer names the net of C2.1, D2.2 (A), D3.2 (A), R1.2, U1.4 (V_{CC}), U1.8 (CE)
- new net: C4.1, L1.2, R4.1, U2.1 (SW)
- new net: Q1.3 (D), R6.2
- new net: J2_SOLAR1.2 (Pin_2), R1.1
